File: esp_button_panel.brd (EAGLE design)
At the start: 50 x 100 mm, 33 parts, among them T1 DMN6068SE-13, T2 DMN6068SE-13, T3 DMN6068SE-13, T4 DMN6068SE-13, U1 V1, U10 V1, U11 V1, U12 V1, U14 V1, U15 V1, U2 V1, U3 V1, U4 V1, U6 V1

Commit message: PCB order version
Parts:
- removed B1: DBL202G, rectifier:DB
- removed D1, D2, D3, D4: ES2D, diode:SMB
- removed RELAY0, RELAY1, RELAY2, RELAY3: SRD-05VDC-SL-C, JKW_CHIP:SRD-05VDC-SL-C
- removed U$2: TEMP-HUM-SENSOR-DHT22, diy-modules:TEMP-HUM-SENSOR-DHT22
- removed U12, U14, U15: V1, JKW_CHIP:2_SCREW_PIN
- added JP1, JP2, JP3: (no value), mylib:2X10
- added LED1, LED2, LED3, LED4: (no value), led:CHIPLED_0805
- added R6, R7, R8: 4k7, rcl:M0805
- added SW1, SW2, SW3, SW4: SKHMPSE010, buttons:SKHMPXE010
- added U5, U7, U8, U9: V1, JKW_CHIP:2_SCREW_PIN
- R1, R2: value 4.7k -> 4k7
- R3, R4, R5: value n.a. -> 4k7
- moved U6 59.0 mm to (5.00, 35.0)
- moved U11 46.9 mm to (5.00, 13.5), turned to 270 degrees
- moved T1 44.8 mm to (19.0, 54.0)
- moved U3 40.5 mm to (45.0, 46.5), turned to 90 degrees
- moved U4 40.0 mm to (45.0, 56.5), turned to 90 degrees
- moved U1 38.5 mm to (5.00, 46.5)
- moved R5 37.8 mm to (11.5, 46.5)
- moved U10 34.5 mm to (45.0, 13.5)
- moved U2 32.5 mm to (5.00, 56.5)
- moved T4 28.4 mm to (31.0, 32.5), turned to 90 degrees
- moved R2 27.4 mm to (31.0, 49.0), turned to 0 degrees
- moved T2 26.0 mm to (31.0, 54.0), turned to 90 degrees
- moved T3 20.8 mm to (19.0, 32.5)
- moved R1 20.6 mm to (19.0, 49.0), turned to 180 degrees
- moved R3 16.1 mm to (19.0, 27.5), turned to 180 degrees
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Connections:
- net RELAY_2 renamed BUTTON_LED_2
- net RELAY_3 renamed BUTTON_LED_3
- removed net +UB: B1.AC1, RELAY0.SWCOMMON, RELAY1.SWCOMMON, RELAY2.SWCOMMON, RELAY3.SWCOMMON, U6.P$1
- removed net -UB: B1.AC2, U1.P$2, U2.P$2, U3.P$2, U4.P$2, U6.P$2
- removed net HUMIDITY: U14.P$1, WEMOS1.A0
- removed net HUMIDITY_P: U12.P$1, WEMOS1.D0
- removed net N$2: B1.+, C3.+, U$3.VIN
- removed net N$8: RELAY3.SWOPEN, U4.P$1
- removed net RELAY_0: R3.2, R4.2, R5.1, T1.1, WEMOS1.D1
- removed net RELAY_1: T2.1, WEMOS1.D2
- removed net RELAY_L_0: D1.A, RELAY0.COIL1, T1.2, T1.4
- removed net RELAY_L_1: D2.A, RELAY1.COIL1, T2.2, T2.4
- removed net RELAY_L_2: D3.A, RELAY2.COIL1, T3.2, T3.4
- removed net RELAY_L_3: D4.A, RELAY3.COIL1, T4.2, T4.4
- removed net SCL: U15.P$2, WEMOS1.D5
- removed net SDA/DHT: R2.1, U$2.2, U15.P$1, WEMOS1.D4
- removed net TEMP: R1.1, U10.P$1, WEMOS1.D6
- new net +12V: C3.+, JP1.10, JP1.2, JP1.4, JP1.6, JP1.8, R5.1, R6.1, R7.1, R8.1, U$3.VIN, U2.P$1, U4.P$2, U6.P$1, U8.P$2, U9.P$2
- new net AIN: JP2.19, JP2.20, U10.P$2
- new net AIN_ESP: JP1.19, JP3.20, WEMOS1.A0
- new net BUTTON_0: R1.2, SW1.1, SW1.2, U1.P$2, WEMOS1.D1
- new net BUTTON_1: R2.2, SW2.1, SW2.2, U3.P$1, WEMOS1.D5
- new net BUTTON_2: R3.2, SW3.1, SW3.2, U5.P$2, WEMOS1.D2
- new net BUTTON_3: R4.2, SW4.1, SW4.2, U7.P$1, WEMOS1.D6
- new net BUTTON_LED_0: T1.1, WEMOS1.D4
- new net BUTTON_LED_1: T2.1, WEMOS1.D8
- new net D0: JP2.1, JP2.2, U11.P$2
- new net D0_ESP: JP1.1, JP3.2, WEMOS1.D0
- new net N$10: LED4.A, R8.2
- new net N$11: LED3.C, T3.2, T3.4, U6.P$2
- new net N$15: LED4.C, T4.2, T4.4, U8.P$1
- new net N$3: LED1.C, T1.2, T1.4, U2.P$2
- new net N$5: LED1.A, R5.2
- net +3V3: now also JP1.12, JP1.14, JP1.16, JP1.18, JP1.20, R1.1, R2.1, R3.1; no longer D1.C, D2.C, D3.C, D4.C, R1.2, R2.2, RELAY0.COIL0, RELAY1.COIL0, RELAY2.COIL0, RELAY3.COIL0, U$2.1, U10.P$2, U11.P$1
- net GND: now also JP3.1, JP3.11, JP3.13, JP3.15, JP3.17, JP3.19, JP3.3, JP3.5, JP3.7, JP3.9, SW1.3, SW1.4, SW1.5, SW2.3, SW2.4, SW2.5, SW3.3, SW3.4, SW3.5, SW4.3, SW4.4, SW4.5, U1.P$1, U10.P$1, U11.P$1, U3.P$2, U5.P$1, U7.P$2, U9.P$1; no longer B1.-, R5.2, U$2.4, U11.P$2, U12.P$2, U14.P$2
- net N$4: now also LED2.A, R6.2; no longer R3.1, RELAY0.SWOPEN, U1.P$1
- net N$6: now also LED3.A, R7.2; no longer RELAY1.SWOPEN, U2.P$1
- net N$7: now also LED2.C, T2.2, T2.4, U4.P$1; no longer RELAY2.SWOPEN, U3.P$1
Routing:
- net +12V: track 0.00 -> 243.6 mm
- net +UB: track 117.3 -> 0.00 mm
- net D0_ESP: track 0.00 -> 108.1 mm, vias 0 -> 1
- net BUTTON_2: track 0.00 -> 106.1 mm
- net SDA/DHT: track 103.8 -> 0.00 mm, vias 1 -> 0
- net -UB: track 103.1 -> 0.00 mm
- net RELAY_0: track 96.8 -> 0.00 mm, vias 2 -> 0
- net BUTTON_3: track 0.00 -> 95.1 mm
- net HUMIDITY_P: track 85.3 -> 0.00 mm, vias 2 -> 0
- net AIN_ESP: track 0.00 -> 85.1 mm, vias 0 -> 1
- net BUTTON_0: track 0.00 -> 79.1 mm
- net HUMIDITY: track 76.3 -> 0.00 mm
- net BUTTON_1: track 0.00 -> 68.1 mm
- net SCL: track 63.2 -> 0.00 mm
- net RELAY_1: track 57.9 -> 0.00 mm, vias 1 -> 0
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Other:
- board text added: "+12V"
- board text added: "+3.3V"
- board text added: "AIN"
- board text added: "BUTTON0"
- board text added: "BUTTON1"
- board text added: "BUTTON2"
- board text added: "BUTTON3"
- board text added: "D0"
- board text added: "ESP Button Panel 2017 MS"
- board text added: "LED0"
- board text added: "LED1"
- board text added: "LED2"
- board text added: "LED3"
- board text removed: "24VAC"
- board text removed: "3.3V"
- board text removed: "ESP 4x RELAY"
- board text removed: "HUM"
- board text removed: "HUM_P"
- board text removed: "MS 2017"
- board text removed: "RELAIS 0"
- board text removed: "RELAIS 1"
- board text removed: "RELAIS 2"
- board text removed: "RELAIS 3"
- board text removed: "SCL"
- board text removed: "SDA"
- board text removed: "TEMP"
