File: esp_button_panel.sch (EAGLE design)
At the start: 33 parts, among them T1 DMN6068SE-13, T2 DMN6068SE-13, T3 DMN6068SE-13, T4 DMN6068SE-13, U1 V1, U10 V1, U11 V1, U12 V1, U14 V1, U15 V1, U2 V1, U3 V1, U4 V1, U6 V1

Commit message: PCB order version
Parts:
- removed B1: DBL202G, rectifier:DBL202G
- removed D1, D2, D3, D4: ES2D, diode:DIODE-SMB
- removed RELAY0, RELAY1, RELAY2, RELAY3: SRD-05VDC-SL-C, JKW_CHIP:RELAYPTH
- removed U$2: TEMP-HUM-SENSOR-DHT22, diy-modules:TEMP-HUM-SENSOR-DHT22
- removed U12, U14, U15: V1, JKW_CHIP:2_PIN_CONNECTOR
- added JP1, JP2, JP3: (no value), mylib:PINHD-2X10
- added LED1, LED2, LED3, LED4: (no value), led:LEDCHIPLED_0805
- added R6, R7, R8: 4k7, rcl:R-EU_M0805
- added SW1, SW2, SW3, SW4: SKHMPSE010, buttons:SKHMPSE010
- added U5, U7, U8, U9: V1, JKW_CHIP:2_PIN_CONNECTOR
- R1, R2: value 4.7k -> 4k7
- R3, R4, R5: value n.a. -> 4k7
Connections:
- net RELAY_2 renamed BUTTON_LED_2
- net RELAY_3 renamed BUTTON_LED_3
- removed net +UB: B1.AC1, RELAY0.SWCOMMON, RELAY1.SWCOMMON, RELAY2.SWCOMMON, RELAY3.SWCOMMON, U6.1
- removed net -UB: B1.AC2, U1.2, U2.2, U3.2, U4.2, U6.2
- removed net HUMIDITY: U14.1, WEMOS1.A0
- removed net HUMIDITY_P: U12.1, WEMOS1.D0
- removed net N$2: B1.+, C3.+, U$3.VIN
- removed net N$8: RELAY3.SWOPEN, U4.1
- removed net RELAY_0: R3.2, R4.2, R5.1, T1.G, WEMOS1.D1
- removed net RELAY_1: T2.G, WEMOS1.D2
- removed net RELAY_L_0: D1.A, RELAY0.COIL1, T1.D
- removed net RELAY_L_1: D2.A, RELAY1.COIL1, T2.D
- removed net RELAY_L_2: D3.A, RELAY2.COIL1, T3.D
- removed net RELAY_L_3: D4.A, RELAY3.COIL1, T4.D
- removed net SCL: U15.2, WEMOS1.D5
- removed net SDA/DHT: R2.1, U$2.DAT, U15.1, WEMOS1.D4
- removed net TEMP: R1.1, U10.1, WEMOS1.D6
- new net +12V: C3.+, JP1.10, JP1.2, JP1.4, JP1.6, JP1.8, R5.1, R6.1, R7.1, R8.1, U$3.VIN, U2.1, U4.2, U6.1, U8.2, U9.2
- new net AIN: JP2.19, JP2.20, U10.2
- new net AIN_ESP: JP1.19, JP3.20, WEMOS1.A0
- new net BUTTON_0: R1.2, SW1.1.1, SW1.1.2, U1.2, WEMOS1.D1
- new net BUTTON_1: R2.2, SW2.1.1, SW2.1.2, U3.1, WEMOS1.D5
- new net BUTTON_2: R3.2, SW3.1.1, SW3.1.2, U5.2, WEMOS1.D2
- new net BUTTON_3: R4.2, SW4.1.1, SW4.1.2, U7.1, WEMOS1.D6
- new net BUTTON_LED_0: T1.G, WEMOS1.D4
- new net BUTTON_LED_1: T2.G, WEMOS1.D8
- new net D0: JP2.1, JP2.2, U11.2
- new net D0_ESP: JP1.1, JP3.2, WEMOS1.D0
- new net N$10: LED4.A, R8.2
- new net N$11: LED3.C, T3.D, U6.2
- new net N$15: LED4.C, T4.D, U8.1
- new net N$3: LED1.C, T1.D, U2.2
- new net N$5: LED1.A, R5.2
- net +3V3: now also JP1.12, JP1.14, JP1.16, JP1.18, JP1.20, R1.1, R2.1, R3.1; no longer D1.C, D2.C, D3.C, D4.C, R1.2, R2.2, RELAY0.COIL0, RELAY1.COIL0, RELAY2.COIL0, RELAY3.COIL0, U$2.VDD, U10.2, U11.1
- net GND: now also JP3.1, JP3.11, JP3.13, JP3.15, JP3.17, JP3.19, JP3.3, JP3.5, JP3.7, JP3.9, SW1.2.1, SW1.2.2, SW1.SH, SW2.2.1, SW2.2.2, SW2.SH, SW3.2.1, SW3.2.2, SW3.SH, SW4.2.1, SW4.2.2, SW4.SH, U1.1, U10.1, U11.1, U3.2, U5.1, U7.2, U9.1; no longer B1.-, R5.2, U$2.GND, U11.2, U12.2, U14.2
- net N$4: now also LED2.A, R6.2; no longer R3.1, RELAY0.SWOPEN, U1.1
- net N$6: now also LED3.A, R7.2; no longer RELAY1.SWOPEN, U2.1
- net N$7: now also LED2.C, T2.D, U4.1; no longer RELAY2.SWOPEN, U3.1
Other:
- note removed: "Will be approx 33.6V!!!"
- moved on the sheet: C3, R1, R2, R3, R4, R5, U1, U10, U11, U2, U3, U4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
